File: Board-Design/Mixed signal Board.kicad_pcb (KiCad board)
At the start: 4 copper layers, 47.1 x 45.7 mm, 92 parts, among them J1 USB_B_Mini, J2 Conn_01x06, J3 USB_B_Mini, J4 Conn_01x04, J5 Conn_01x04, J6 Terminal Block 2.5mm, Q1 MMBT3904, SW1 TACTILE SWITCH, SW2 TACTILE SWITCH, U1 STM32F103C8Tx, U2 CH340C, U3 MMICT5848-00-012, U4 SHT40-AD1B-R2, U5 SGP40-D-R4, U6 STM32F407VGTx, U7 LD1117S33TR_SOT223, U8 LD1117S18TR_SOT223, X1 8MHZ, X2 8MHZ

Commit message: Add files via upload
Parts:
- C31, C32: moved to F.Cu
- moved C32 0.90 mm to (-106.3, 71.2)
- moved C31 0.81 mm to (-117.6, 71.2)
Connections:
- H2 pad 1: unconnected-(H2-Pad1) -> GND
- H4 pad 1: unconnected-(H4-Pad1) -> GND
Routing:
- net GND: track 110.7 -> 95.5 mm
- net +3V3: track 57.2 -> 58.7 mm
- net NTRST_F407: track 39.3 -> 38.1 mm
- net I2C_SCL: track 38.4 -> 37.1 mm
- net I2C_SDA: track 32.3 -> 33.3 mm
Other:
- board size 47.1 x 45.7 mm -> 47.1 x 45.3 mm
